File: CAD_data/SO2R-Controler-shield-v1r1_0/HeadphoneSwitch.sch (KiCad schematic (older format))
At the start: 71 parts, among them IC1 AE-PCA9306, U1 ARDUINOR3-BPLACE

Commit message: CAD_data
Connections:
- wire segments 151 -> 149
Changed lines of the file:
@@
 	1300 4550 1600 4550
-Wire Wire Line
-	1300 4750 1800 4750
-Wire Wire Line
-	1300 4950 3000 4950
 Wire Wire Line
 	5450 6350 5900 6350
@@
 Text Label 6100 6550 0    10   ~ 0
 GND1
-Wire Wire Line
-	1800 4750 1800 5450
 Text Label 1800 4750 0    10   ~ 0
 GND1
-Wire Wire Line
-	3000 5450 3000 4950
 Text Label 3000 5450 0    10   ~ 0
 GND1
@@
 	1    0    0    -1
 $EndComp
-Connection ~ 1800 4750
-Wire Wire Line
-	1800 4750 2800 4750
-Connection ~ 3000 4950
-Wire Wire Line
-	3000 4950 3200 4950
+Wire Wire Line
+	1800 4750 1800 5450
+Wire Wire Line
+	1300 4750 2800 4750
+Wire Wire Line
+	3000 5450 3000 4950
+Wire Wire Line
+	1300 4950 3200 4950
 Wire Bus Line
 	5600 1650 5600 5050

Commit message: CAD_data
Connections:
- wire segments 149 -> 152
- no-connect marks 0 -> 5
Changed lines of the file:
@@
 Wire Wire Line
 	1300 4950 3200 4950
+NoConn ~ 4900 1350
+NoConn ~ 4900 1450
+NoConn ~ 4900 1550
+NoConn ~ 2500 1950
+NoConn ~ 2500 1850
+$Comp
+L HeadphoneSwitch-eagle-import:VCC #SUPPLY0101
+U 1 0 5C041CF0
+P 9950 3950
+F 0 "#SUPPLY0101" H 9950 3950 50  0001 C CNN
+F 1 "VCC" H 9875 4075 59  0000 L BNN
+F 2 "" H 9950 3950 50  0001 C CNN
+F 3 "" H 9950 3950 50  0001 C CNN
+	1    9950 3950
+	1    0    0    -1
+$EndComp
+$Comp
+L power:PWR_FLAG #FLG0101
+U 1 1 5C041D90
+P 9950 4200
+F 0 "#FLG0101" H 9950 4275 50  0001 C CNN
+F 1 "PWR_FLAG" H 9950 4373 50  0000 C CNN
+F 2 "" H 9950 4200 50  0001 C CNN
+F 3 "~" H 9950 4200 50  0001 C CNN
+	1    9950 4200
+	-1   0    0    1
+$EndComp
+Wire Wire Line
+	9950 4200 9950 4050
+$Comp
+L HeadphoneSwitch-eagle-import:+3V3 #+3V0101
+U 1 0 5C04A7E5
+P 10400 3850
+F 0 "#+3V0101" H 10400 3850 50  0001 C CNN
+F 1 "+3V3" V 10300 3650 59  0000 L BNN
+F 2 "" H 10400 3850 50  0001 C CNN
+F 3 "" H 10400 3850 50  0001 C CNN
+	1    10400 3850
+	1    0    0    -1
+$EndComp
+$Comp
+L power:PWR_FLAG #FLG0102
+U 1 1 5C04A99B
+P 10400 4200
+F 0 "#FLG0102" H 10400 4275 50  0001 C CNN
+F 1 "PWR_FLAG" H 10400 4373 50  0000 C CNN
+F 2 "" H 10400 4200 50  0001 C CNN
+F 3 "~" H 10400 4200 50  0001 C CNN
+	1    10400 4200
+	-1   0    0    1
+$EndComp
+Wire Wire Line
+	10400 4200 10400 3950
+$Comp
+L HeadphoneSwitch-eagle-import:GND1 #SUPPLY0102
+U 1 0 5C051906
+P 10800 4250
+F 0 "#SUPPLY0102" H 10800 4250 50  0001 C CNN
+F 1 "GND1" H 10715 4125 59  0000 L BNN
+F 2 "" H 10800 4250 50  0001 C CNN
+F 3 "" H 10800 4250 50  0001 C CNN
+	1    10800 4250
+	1    0    0    -1
+$EndComp
+$Comp
+L power:PWR_FLAG #FLG0103
+U 1 1 5C057DF8
+P 10800 3950
+F 0 "#FLG0103" H 10800 4025 50  0001 C CNN
+F 1 "PWR_FLAG" H 10800 4124 50  0000 C CNN
+F 2 "" H 10800 3950 50  0001 C CNN
+F 3 "~" H 10800 3950 50  0001 C CNN
+	1    10800 3950
+	1    0    0    -1
+$EndComp
+Wire Wire Line
+	10800 3950 10800 4150
 Wire Bus Line
 	5600 1650 5600 5050
